File: Welding.sch (KiCad schematic (older format))
At the start: 19 parts, among them Q1 PSMN0R9-30YLD, Q2 PSMN0R9-30YLD, Q3 PSMN0R9-30YLD, Q4 PSMN0R9-30YLD, Q5 PSMN0R9-30YLD, Q6 PSMN0R9-30YLD, U5 FAN3111CSX

Commit message: Layout finish
Parts:
- removed U5: FAN3111CSX, Package_TO_SOT_SMD:SOT-23-5_HandSoldering, symbol microSpot:FAN3111
- added C7, C8: 1n, Capacitor_SMD:C_0805_2012Metric_Pad1.15x1.40mm_HandSolder, symbol Device:C
- added D6, D7: BZX84C3V3, Package_TO_SOT_SMD:SOT-23, symbol Device:D_Zener
- added R14, R23: 5k, Resistor_SMD:R_0805_2012Metric_Pad1.15x1.40mm_HandSolder, symbol Device:R
- added R22, R24: 1k8, Resistor_SMD:R_0805_2012Metric_Pad1.15x1.40mm_HandSolder, symbol Device:R
- added U4: FAN3111E, Package_TO_SOT_SMD:SOT-23-5_HandSoldering, symbol MicroSpot~v2:FAN3111E
- C12: footprint Capacitor_SMD:C_1206_3216Metric_Pad1.42x1.75mm_HandSolder -> Capacitor_SMD:C_0805_2012Metric_Pad1.15x1.40mm_HandSolder
- R12: value 10k -> 5k; footprint Resistor_SMD:R_1206_3216Metric_Pad1.42x1.75mm_HandSolder -> Resistor_SMD:R_0805_2012Metric_Pad1.15x1.40mm_HandSolder
- R13, R15, R16, R17, R18, R19, R20, R21, TH1: footprint Resistor_SMD:R_1206_3216Metric_Pad1.42x1.75mm_HandSolder -> Resistor_SMD:R_0805_2012Metric_Pad1.15x1.40mm_HandSolder
Connections:
- net labels added: WELD+, WELD-
- net labels removed: +5V
- wire segments 74 -> 96
Other:
- moved on the sheet: C12, D5, R12, R13, R16, TH1

Commit message: Changes FAN3111 footprint and removed 5V
Connections:
- net labels added: +3V3
- net labels removed: +3.3V
- wire segments 96 -> 97
Changed lines of the file:
@@
 	0    1    1    0
-$EndComp
-$Comp
-L power:+3.3V #PWR0118
-U 1 1 5EE03885
-P 7250 4550
-F 0 "#PWR0118" H 7250 4400 50  0001 C CNN
-F 1 "+3.3V" H 7265 4723 50  0000 C CNN
-F 2 "" H 7250 4550 50  0001 C CNN
-F 3 "" H 7250 4550 50  0001 C CNN
-	1    7250 4550
-	1    0    0    -1
 $EndComp
 Wire Wire Line
@@
 	2900 2725 2900 2650
 $Comp
-L power:+3.3V #PWR?
-U 1 1 603D0425
+L power:+3V3 #PWR?
+U 1 1 604236BB
 P 2900 2650
 F 0 "#PWR?" H 2900 2500 50  0001 C CNN
-F 1 "+3.3V" H 2915 2823 50  0000 C CNN
+F 1 "+3V3" H 2915 2823 50  0000 C CNN
 F 2 "" H 2900 2650 50  0001 C CNN
 F 3 "" H 2900 2650 50  0001 C CNN
@@
 	1    0    0    -1
 $EndComp
+$Comp
+L power:+3V3 #PWR?
+U 1 1 60423D14
+P 7250 4475
+F 0 "#PWR?" H 7250 4325 50  0001 C CNN
+F 1 "+3V3" H 7265 4648 50  0000 C CNN
+F 2 "" H 7250 4475 50  0001 C CNN
+F 3 "" H 7250 4475 50  0001 C CNN
+	1    7250 4475
+	1    0    0    -1
+$EndComp
+Wire Wire Line
+	7250 4550 7250 4475
 $EndSCHEMATC
